File: apps/rdc/hardware/hardware_project/Phase Splitter.kicad_sch (KiCad schematic)
At the start: 48 parts, among them Q1 BC817, Q2 BC817, Q3 BC807, Q4 BC807, Q5 BC817, Q6 BC807, Q7 BC817, Q8 BC807, Q9 BC817, T16 EXC_N, T17 EXC_P, U1 TLV4171IPWR

Commit message: hpm apps release v1.8.0
Signed-off-by: zhangeg <engui.zhang@hpmicro.com>
Other:
- moved on the sheet: C9, R19, R24, R25, R26, R27, U1D
