File: apps/adc/hardware/HPM6P00ADCEVKRevB-工程文件/HPM6P00ADCEVKRevB/ADC_Signal.kicad_sch (KiCad schematic)
At the start: 96 parts

Commit message: hpm apps release v1.11.0
Signed-off-by: zhangeg <engui.zhang@hpmicro.com>
Parts:
- renumbered W6 to W8
Other:
- title: HPM6P00EVKRevB -> HPM6P00ADCEVKRevB
