File: apps/adc/hardware/HPM6P00ADCEVKRevB-工程文件/HPM6P00ADCEVKRevB/Assembly.kicad_sch (KiCad schematic)
At the start: 4 parts

Commit message: hpm apps release v1.11.0
Signed-off-by: zhangeg <engui.zhang@hpmicro.com>
Other:
- title: HPM6P00EVKRevB -> HPM6P00ADCEVKRevB
