File: apps/adc/hardware/HPM6P00ADCEVKRevB-工程文件/HPM6P00ADCEVKRevB/HPM6P00ADCEVKRevB.kicad_sch (KiCad schematic)
At the start: 0 parts

Commit message: hpm apps release v1.11.0
Signed-off-by: zhangeg <engui.zhang@hpmicro.com>
Other:
- removed sheet ADC_Signal_IN
- removed sheet Assembly
- removed sheet DEBUG
- removed sheet MCU_PA&JTAG&FLASH
- removed sheet MCU_PB&PC
- removed sheet MCU_PD
- removed sheet MCU_POWER
- removed sheet MCU_PY
- removed sheet MCU_USB&OSC
- removed sheet Power
- removed sheet SDM
- removed sheet Signal_Power
- removed sheet USB
- removed sheet VREF
- added sheet HPM6P00ADCEVK MAINENTRY (HPM6P00ADCEVK MAINENTRY.kicad_sch)
- note added: "20241013"
- note added: "Diff ADC x1"
- note added: "FLASH"
- note added: "HPM6P00"
- note added: "HPM6P00ADCEVKRevB"
- note added: "JTAG20PIN"
- note added: "POWER"
- note added: "SDM x4"
- note added: "Single ADC x4"
- note added: "System Block Diagram"
- note added: "USB TYPE C"
- note added: "USB转UART"
- note added: "修订历史"
- note added: "内容"
- note added: "时间"
- title: HPM600EVK_RevA -> HPM6P00EVKRevB
