File: apps/adc/hardware/HPM6P00ADCEVKRevB-工程文件/HPM6P00ADCEVKRevB/MCU_PB&PC.kicad_sch (KiCad schematic)
At the start: 7 parts, among them U14 HPM600

Commit message: hpm apps release v1.11.0
Signed-off-by: zhangeg <engui.zhang@hpmicro.com>
Parts:
- renumbered U14 to U9
Other:
- title: HPM6P00EVKRevB -> HPM6P00ADCEVKRevB
