File: apps/adc/hardware/HPM6P00ADCEVKRevB-工程文件/HPM6P00ADCEVKRevB/SDM.kicad_sch (KiCad schematic)
At the start: 1 part, among them J4 HEADER 5X2

Commit message: hpm apps release v1.11.0
Signed-off-by: zhangeg <engui.zhang@hpmicro.com>
Other:
- title: HPM6P00EVKRevB -> HPM6P00ADCEVKRevB
