File: apps/adc/hardware/HPM6P00ADCEVKRevB-工程文件/HPM6P00ADCEVKRevB/USB.kicad_sch (KiCad schematic)
At the start: 22 parts, among them U2 PW1515

Commit message: hpm apps release v1.11.0
Signed-off-by: zhangeg <engui.zhang@hpmicro.com>
Parts:
- D?: value 1N5819HW-7-F -> 1N5819HW-7-F
- renumbered C143 to C1
Other:
- title: HPM6P00EVKRevB -> HPM6P00ADCEVKRevB
